File: HeleSystemet.kicad_sch (KiCad schematic)
At the start: 19 parts, among them U1 SX1276, U2 ADA4898-1YRDZ

Commit message: Add files via upload
Parts:
- removed D1: D, symbol Device:D
- removed Spændingsregulator: L7805, symbol Regulator_Linear:L7805
- added C2: 100μF, symbol Device:C
- added C3: 470μF, symbol Device:C
- added D3: 1N5822, Diode_THT:D_DO-201AD_P15.24mm_Horizontal, symbol Diode:1N5822
- added L1: 680μH, symbol Device:L
- added U3: LM358, symbol Amplifier_Operational:LM358
- added U4: LM2575-5.0BT, Package_TO_SOT_THT:TO-220-5_Vertical, symbol Regulator_Switching:LM2575-5.0BT
- A1: value Arduino_UNO_R3 -> Arduino
- HavbøjensBat: value 18 V -> 9-25 V
- R2: value 8.8MΩ -> 10MΩ
- R3, R4: value 150K -> 44K
- renumbered 0.15 to 0.47
Connections:
- net 5V is gone; now on net GND: U2.7 (V+), U2.8 (~{PD})
- net 3V3: no longer A1.4 (3V3)
- net D8: now also R4.2; no longer R3.1
- net GND: now also 0.47.1, 0.47.2, HavbøjensBat.1 (+), LA1.2 (+), R1.1, R2.1, R2.2, R3.1, C2.1, C2.2, C3.2, D3.2 (A), U4.1 (VIN), U4.3 (GND), U4.5 (~{ON}/OFF); no longer R4.2
- net at R2.1, R3.2: now also U3.3 (+); no longer A1.11 (A2)
- net at A1.13 (SDA/A4): no longer Accelorometer.24 (SDA)
- net at A1.14 (SCL/A5): no longer Accelorometer.23 (SCL)
- net at A1.31 (SDA/A4): now also Accelorometer.24 (SDA)
- net at A1.32 (SCL/A5): now also Accelorometer.23 (SCL)
- net at A1.5 (+5V), Accelorometer.13 (VDD), D2.1 (K)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: now also C3.1, L1.2, U4.4 (FB)
- new net: A1.11 (A2), U3.1, U3.2 (-)
- new net: D3.1 (K), L1.1, U4.2 (OUT)
- new net VCC: A1.4 (3V3)
Other:
- moved on the sheet: 0.47, GPS, HavbøjensBat, LA1, R1, R2, R3, R4, U2
